File: Thorlabs 30 mm Cage Plate LED MCPCB/Thorlabs 30 mm Cage Plate LED MCPCB.kicad_pcb (KiCad board)
At the start: 2 copper layers, 40 x 40 mm, 4 parts

Commit message: Rats nest connected
Parts:
- added C1: 10μF, Capacitor_SMD:C_0603_1608Metric, F.Cu at (109.8, 83.1)
- added D1: LED, Custom:LED_SST-20-DR, F.Cu at (120.0, 80.0)
- added D2: D_Schottky, Custom:D_SOD-128, F.Cu at (110.3, 78.1)
- added IC1: AL8843QSP-13, Custom:SO-8EP_3P9X4P95_DIO, F.Cu at (105.1, 81.2)
- added J2: Conn_01x04, Custom:SAMTEC_SSM-104-L-SH, F.Cu at (120.0, 93.7)
- added L1: 47μH, Custom:SRP1038A-220M_BRN, F.Cu at (119.9, 65.2)
- added R1: 0.05, Resistor_SMD:R_1206_3216Metric, F.Cu at (110.2, 73.8)
Routing:
- net GND: track 0.00 -> 60.8 mm
- net Net-(D1-A): track 0.00 -> 51.5 mm
- net /Vin: track 0.00 -> 27.1 mm
- net Net-(D2-A): track 0.00 -> 18.8 mm
- net Net-(D1-K): track 0.00 -> 15.9 mm
- net /PWM: track 0.00 -> 14.3 mm

Commit message: Full working draft
Parts:
- added C2: 10μF, Capacitor_SMD:C_0603_1608Metric, F.Cu at (111.3, 83.1)
- added C3: 10μF, Capacitor_SMD:C_0603_1608Metric, F.Cu at (112.8, 83.1)
- added REF**: CC-BY-SA Symbol, Custom:CC-BY-SA Symbol, F.Cu at (109.7, 88.1)
- added REF**: OSHW-Logo_5.7x6mm_SilkScreen, Symbol:OSHW-Logo_5.7x6mm_SilkScreen, F.Cu at (111.5, 94.7)
- renumbered D2 to D1, D1 to D2
Routing:
- net Net-(D2-K): track 15.9 -> 20.9 mm
- net Net-(D2-A): track 51.5 -> 49.8 mm
- net /PWM: track 14.3 -> 13.5 mm
- added copper zone on F.Cu, net /Vin
- added copper zone on F.Cu, net GND
- added copper zone on F.Cu, net Net-(D1-A)
- added copper zone on F.Cu, net Net-(D2-A)
- added copper zone on F.Cu, net Net-(D2-K)
Other:
- board text added: "30mm Cage Plate LED Driver"
- board text added: "Designed by: Benjamin E. Smith Funded by: NIH P30EY003176 https://github.com/Llamero/ 30mm_cage_plate_LED_MCPCB"
- board text added: "Gnd Ctrl Vin Gnd"

Commit message: PCB optimization
Parts:
- renumbered J2 to J1
Routing:
- net Net-(D2-A): track 49.8 -> 54.4 mm
- net Net-(D2-K): track 20.9 -> 21.7 mm
Other:
- board text added: "30 mm Cage Plate LED Driver"
- board text removed: "30mm Cage Plate LED Driver"
Changed lines of the file:
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@@
   (setup
     (pad_to_mask_clearance 0)
+    (grid_origin 111.76 63.5)
     (pcbplotparams
       (layerselection 0x00010fc_ffffffff)
@@
     (property "ki_keywords" "connector")
     (attr smd)
-    (fp_text reference "J2" (at -6.1 -0.21) (layer "F.SilkS")
+    (fp_text reference "J1" (at -6.1 -0.21) (layer "F.SilkS")
         (effects (font (size 1 1) (thickness 0.15)))
     )
@@
         (effects (font (size 1 1) (thickness 0.15)))
     )
-    (fp_text user "-" (at 1.98 0.51 180 unlocked) (layer "F.SilkS")
+    (fp_text user "-" (at -3.2 0.5 180 unlocked) (layer "F.SilkS")
         (effects (font (size 1 1) (thickness 0.1)) (justify left bottom))
     )
-    (fp_text user "+" (at -3.31 0.51 180 unlocked) (layer "F.SilkS")
+    (fp_text user "+" (at 1.9 0.51 180 unlocked) (layer "F.SilkS")
         (effects (font (size 1 1) (thickness 0.1)) (justify left bottom))
     )
@@
     (property "ki_keywords" "capacitor cap")
     (attr smd)
-    (fp_text reference "C1" (at -2.30495 -0.25 180) (layer "F.SilkS")
+    (fp_text reference "C1" (at -2.28495 -0.28 180) (layer "F.SilkS")
         (effects (font (size 1 1) (thickness 0.15)))
     )
@@
   (gr_line (start 100 62) (end 102 60)
     (stroke (width 0.1) (type default)) (layer "Edge.Cuts"))
-  (gr_text "30mm Cage Plate LED Driver" (at 131.64 93.46 90) (layer "F.SilkS")
+  (gr_text "30 mm Cage Plate LED Driver" (at 131.5 94 90) (layer "F.SilkS")
     (effects (font (size 1.2 1.2) (thickness 0.2) bold) (justify left bottom))
   )
@@
   (segment (start 115.831001 67.288999) (end 110.3351 72.7849) (width 1) (layer "F.Cu") (net 3))
   (segment (start 107.8051 79.32005) (end 107.8051 80.59005) (width 1) (layer "F.Cu") (net 3))
+  (segment (start 118.71 67.55) (end 118.7 67.54) (width 2) (layer "F.Cu") (net 4))
+  (segment (start 112.77 63.05) (end 112.77 62.99) (width 1.5) (layer "F.Cu") (net 4))
+  (segment (start 115.56 62.2) (end 118.86 62.2) (width 1.5) (layer "F.Cu") (net 4))
+  (segment (start 113.36 62.4) (end 113.56 62.2) (width 1.5) (layer "F.Cu") (net 4))
   (segment (start 104.77 73.82495) (end 108.7775 73.82495) (width 0.5) (layer "F.Cu") (net 4))
   (segment (start 118.71 76.97) (end 118.73 76.99) (width 2) (layer "F.Cu") (net 4))
+  (segment (start 118.86 62.2) (end 118.86 71.5) (width 1.5) (layer "F.Cu") (net 4))
   (segment (start 101.1956 81.41005) (end 101.1956 77.39935) (width 0.5) (layer "F.Cu") (net 4))
   (segment (start 118.6157 80) (end 118.6157 77.7657) (width 0.5) (layer "F.Cu") (net 4))
   (segment (start 108.7775 73.82495) (end 108.7775 70.4925) (width 1) (layer "F.Cu") (net 4))
-  (segment (start 118.71 62.56) (end 118.71 76.97) (width 2) (layer "F.Cu") (net 4))
   (segment (start 118.6157 77.7657) (end 118.61 77.76) (width 0.5) (layer "F.Cu") (net 4))
-  (segment (start 118.5506 62.4006) (end 113.4194 62.4006) (width 2) (layer "F.Cu") (net 4))
-  (segment (start 118.71 62.56) (end 118.5506 62.4006) (width 2) (layer "F.Cu") (net 4))
+  (segment (start 108.7775 67.0425) (end 112.77 63.05) (width 2) (layer "F.Cu") (net 4))
+  (segment (start 118.71 76.97) (end 118.71 67.55) (width 2) (layer "F.Cu") (net 4))
   (segment (start 102.3949 81.86005) (end 101.6456 81.86005) (width 0.5) (layer "F.Cu") (net 4))
   (segment (start 101.6456 81.86005) (end 101.1956 81.41005) (width 0.5) (layer "F.Cu") (net 4))
+  (segment (start 112.77 62.99) (end 113.36 62.4) (width 1.5) (layer "F.Cu") (net 4))
   (segment (start 101.1956 77.39935) (end 104.77 73.82495) (width 0.5) (layer "F.Cu") (net 4))
-  (segment (start 113.4194 62.4006) (end 108.7775 67.0425) (width 2) (layer "F.Cu") (net 4))
   (segment (start 108.7775 70.4925) (end 108.7775 67.0425) (width 2) (layer "F.Cu") (net 4))
+  (segment (start 113.56 62.2) (end 115.56 62.2) (width 1.5) (layer "F.Cu") (net 4))
   (segment (start 118.257462 88.19) (end 113.197512 83.13005) (width 0.2) (layer "F.Cu") (net 6))
   (segment (start 118.66 88.6575) (end 118.66 88.19) (width 0.2) (layer "F.Cu") (net 6))
@@
   (segment (start 118.74 88.7375) (end 118.66 88.6575) (width 0.2) (layer "F.Cu") (net 6))
   (segment (start 118.66 88.19) (end 118.257462 88.19) (width 0.2) (layer "F.Cu") (net 6))
-  (segment (start 120.91 65.2) (end 120.91 76.29) (width 2) (layer "F.Cu") (net 7))
-  (segment (start 120.91 76.29) (end 121.08 76.46) (width 2) (layer "F.Cu") (net 7))
+  (segment (start 121.3843 65.2843) (end 121.3843 80) (width 2) (layer "F.Cu") (net 7))
   (segment (start 120 80) (end 121.08 78.92) (width 1) (layer "F.Cu") (net 7))
-  (segment (start 120.96 65.15) (end 120.91 65.2) (width 2) (layer "F.Cu") (net 7))
-  (segment (start 124.028999 65.15) (end 120.96 65.15) (width 2) (layer "F.Cu") (net 7))
+  (segment (start 121.25 65.15) (end 121.3843 65.2843) (width 2) (layer "F.Cu") (net 7))
+  (segment (start 124.028999 65.15) (end 121.25 65.15) (width 2) (layer "F.Cu") (net 7))
   (segment (start 121.3843 80) (end 121.3843 77.5757) (width 0.5) (layer "F.Cu") (net 7))
   (segment (start 121.3843 77.5757) (end 121.4 77.56) (width 0.5) (layer "F.Cu") (net 7))
-  (segment (start 121.08 78.92) (end 121.08 76.46) (width 1) (layer "F.Cu") (net 7))
   (zone (net 1) (net_name "GND") (layer "F.Cu") (hatch edge 0.5)
     (connect_pads yes (clearance 0.5))
@@
         (xy 140.09 100)
         (xy 99.99 100.04)
+      )
+    )
+  )
+  (zone (net 4) (net_name "Net-(D2-A)") (layer "F.Cu") (hatch edge 0.5)
+    (priority 5)
+    (connect_pads yes (clearance 0.5))
+    (min_thickness 0.25) (filled_areas_thickness no)
+    (fill yes (thermal_gap 0.5) (thermal_bridge_width 0.5))
+    (polygon
+      (pts
+        (xy 119 76.96)
+        (xy 117.71 76.93)
+        (xy 117.71 81.71)
+        (xy 119 81.75)
       )
     )
@@
       (pts
         (xy 118.97 65.98)
-        (xy 118.97 81.94)
-        (xy 116.98 81.71)
-        (xy 114.62 72.88)
+        (xy 118.55 72.98)
         (xy 110.34 72.91)
         (xy 115.78 67.33)
@@
         (xy 111.65 76.56)
         (xy 111.62 72.88)
-        (xy 114.62 72.88)
-        (xy 116.431783 79.658833)
-        (xy 116.98 81.71)
+        (xy 118.55 72.98)
+        (xy 118.57 83.22)
         (xy 123.41 88.1)
+      )
+    )
+  )
+  (zone (net 3) (net_name "Net-(D1-A)") (layer "F.Cu") (hatch edge 0.5)
+    (priority 6)
+    (connect_pads yes (clearance 0.5))
+    (min_thickness 0.25) (filled_areas_thickness no)
+    (fill yes (thermal_gap 0.5) (thermal_bridge_width 0.5))
+    (polygon
+      (pts
+        (xy 110.34 75.78)
+        (xy 106.95 75.78)
+        (xy 106.9 81.07)
+        (xy 108.72 81.08)
+        (xy 108.72 79.34)
+        (xy 111.32 76.6)
       )
     )
@@
     (polygon
       (pts
-        (xy 108.56 72.62)
+        (xy 107.87 72.89)
         (xy 110.58 72.66)
         (xy 115.78 67.33)
-        (xy 115.94 63.67)
-        (xy 112.39 63.67)
-        (xy 108.79 66.88)
+        (xy 119.7 67.31)
+        (xy 119.67 61.42)
+        (xy 112.98 61.42)
+        (xy 107.8 66.57)
       )
     )
@@
     (polygon
       (pts
-        (xy 118.43 61.45)
+        (xy 119.67 61.42)
         (xy 137.23 61.36)
         (xy 137.21 98.56)
