File: Thorlabs 30 mm Cage Plate LED MCPCB/Thorlabs 30 mm Cage Plate LED MCPCB.kicad_sch (KiCad schematic)
At the start: 10 parts, among them IC1 AL8843QSP-13, J2 Conn_01x04

Commit message: Rats nest connected
Parts:
- added D2: D_Schottky, Custom:D_SOD-128, symbol Device:D_Schottky
- C1: renamed from C2; value C_Small -> 10μF; footprint (none) -> Capacitor_SMD:C_0603_1608Metric; Manufacturer (none) -> Murata Electronics; Part (none) -> GRM188R6YA106MA73D
- D1: footprint (none) -> Custom:LED_SST-20-DR; Manufacturer (none) -> Luminus Devices Inc.; Part (none) -> SST-20-DR-B120H-AA660
- J2: footprint (none) -> Custom:SAMTEC_SSM-104-L-SH; Manufacturer (none) -> SSM-104-F-SH-TR; Part (none) -> SSM-104-F-SH-TR
- L1: value L -> 47μH; footprint (none) -> Custom:SRP1038A-220M_BRN; Manufacturer (none) -> Bourns Inc.; Part (none) -> SRP1038A-470M
- R1: value R -> 0.05; footprint (none) -> Resistor_SMD:R_1206_3216Metric; Manufacturer (none) -> Ohmite; Part (none) -> MCS1632R050FER
Connections:
- net GND: now also J2.1 (Pin_1); no longer J2.2 (Pin_2)
- net Vin: now also J2.2 (Pin_2), D2.1 (K); no longer J2.1 (Pin_1)
- net at IC1.7 (SW), IC1.8 (SW), L1.2: now also D2.2 (A)
Other:
- moved on the sheet: J2

Commit message: Full working draft
Parts:
- added C2, C3: 10μF, Capacitor_SMD:C_0603_1608Metric, symbol Device:C_Small
- renumbered D2 to D1, D1 to D2
Connections:
- net GND: now also C2.1, C3.1
- net Vin: now also C2.2, C3.2
Other:
- moved on the sheet: J2

Commit message: PCB optimization
Parts:
- renumbered J2 to J1
Changed lines of the file:
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@@
   (symbol (lib_id "Connector_Generic:Conn_01x04") (at 125.73 48.26 0) (unit 1)
     (in_bom yes) (on_board yes) (dnp no) (fields_autoplaced)
-    (property "Reference" "J2" (at 128.27 48.26 0)
+    (property "Reference" "J1" (at 128.27 48.26 0)
       (effects (font (size 1.27 1.27)) (justify left))
     )
@@
       (project "Thorlabs 30 mm Cage Plate LED MCPCB"
         (path "/d4bfa918-6f2d-41e7-978b-b2160bded453"
-          (reference "J2") (unit 1)
+          (reference "J1") (unit 1)
         )
       )
