File: KiCAD/30 mm Cage Plate LED MCPCB.kicad_pcb (KiCad board)
At the start: 2 copper layers, 70.5 x 70.5 mm, 22 parts, among them IC1 AL8843QSP-13, J1 8P8C_Shielded

Commit message: Add T-cube connectivity
Connections:
- D2 pad 1: Net-(IC1-SET) -> /LED+
- D2 pad 8: Net-(D2-PAD) -> /LED-
- D2 pad 9: Net-(D2-PAD) -> /LED-
- IC1 pad 3: Net-(IC1-SET) -> /LED+
- J1 pad 3: /Vin -> /LED+
- J1 pad 4: GND -> /LED-
- L1 pad 1: Net-(D2-PAD) -> /LED-
- R1 pad 1: Net-(IC1-SET) -> /LED+
Routing:
- net /LED-: track 0.00 -> 31.1 mm
- net /LED+: track 0.00 -> 24.9 mm
- net /Vin: track 17.3 -> 13.6 mm
- net GND: track 52.1 -> 48.5 mm
- net Net-(IC1-SET): track 2.06 -> 0.00 mm
- added copper zone on F.Cu, net /LED+
- added copper zone on F.Cu, net /LED-
- removed copper zone on F.Cu, net Net-(D2-PAD)
- removed copper zone on F.Cu, net Net-(IC1-SET)
Other:
- board text added: "Ctrl Vin LED Temp"
- board text removed: "Ctrl Vled Vled Temp"
Changed lines of the file:
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@@
 	(net 3 "Net-(D1-A)")
 	(net 4 "unconnected-(IC1-NC-Pad4)")
-	(net 5 "Net-(D2-PAD)")
+	(net 5 "/LED-")
 	(net 6 "Net-(D2-A-Pad3)")
 	(net 7 "Net-(D2-A-Pad5)")
 	(net 8 "Net-(D2-A-Pad7)")
-	(net 9 "Net-(IC1-SET)")
+	(net 9 "/LED+")
 	(net 10 "/CTRL")
 	(net 11 "/Temp")
@@
 			(layers "F.Cu" "F.Paste" "F.Mask")
 			(roundrect_rratio 0.2222222222)
-			(net 9 "Net-(IC1-SET)")
+			(net 9 "/LED+")
 			(pintype "passive")
 		)
@@
 			(layers "F.Cu" "F.Paste" "F.Mask")
 			(roundrect_rratio 0.25)
-			(net 2 "/Vin")
+			(net 9 "/LED+")
 			(pintype "passive")
 			(thermal_bridge_angle 45)
@@
 			(layers "F.Cu" "F.Paste" "F.Mask")
 			(roundrect_rratio 0.25)
-			(net 1 "GND")
+			(net 5 "/LED-")
 			(pintype "passive")
 			(thermal_bridge_angle 45)
@@
 			(size 1.4986 0.5588)
 			(layers "F.Cu" "F.Paste" "F.Mask")
-			(net 9 "Net-(IC1-SET)")
+			(net 9 "/LED+")
 			(pinfunction "SET")
 			(pintype "unspecified")
@@
 		(tags "resistor")
 		(property "Reference" "TH1"
-			(at -0.11 1.44 360)
+			(at -0.11 1.44 0)
 			(layer "F.SilkS")
 			(effects
@@
 		)
 		(property "Value" "Thermistor"
-			(at 0 1.43 360)
+			(at 0 1.43 0)
 			(layer "F.Fab")
 			(effects
@@
 		)
 		(fp_text user "${REFERENCE}"
-			(at 0 0 360)
+			(at 0 0 0)
 			(layer "F.Fab")
 			(effects
@@
 			(size 3.302 3.0988)
 			(layers "F.Cu" "F.Paste" "F.Mask")
-			(net 5 "Net-(D2-PAD)")
+			(net 5 "/LED-")
 			(pinfunction "1")
 			(pintype "passive")
@@
 			)
 		)
-		(property "Datasheet" "LZ4-00"
+		(property "Datasheet" "https://look.ams-osram.com/m/60f2d29fa455f5ac/original/LZ4-00R308.pdf"
 			(at 0 0 90)
 			(unlocked yes)
@@
 			(chamfer_ratio 0.28)
 			(chamfer bottom_right)
-			(net 9 "Net-(IC1-SET)")
+			(net 9 "/LED+")
 			(pinfunction "A")
 			(pintype "passive")
@@
 			(size 1.16 1.16)
 			(layers "F.Cu" "F.Paste" "F.Mask")
-			(net 5 "Net-(D2-PAD)")
+			(net 5 "/LED-")
 			(pinfunction "K")
 			(pintype "passive")
@@
 			(size 4.64 4.64)
 			(layers "F.Cu" "F.Paste" "F.Mask")
-			(net 5 "Net-(D2-PAD)")
+			(net 5 "/LED-")
 			(pinfunction "PAD")
 			(pintype "passive")
@@
 		)
 	)
-	(gr_text "Ctrl\nVled\nVled\nTemp"
+	(gr_text "Ctrl\nVin\nLED\nTemp"
 		(at 0 18.18 90)
 		(layer "F.SilkS")
@@
 	)
 	(segment
-		(start 3.17 22.79)
-		(end 3.93 22.79)
+		(start -3.5078 4.7178)
+		(end -4.8 4.7178)
 		(width 0.25)
 		(layer "F.Cu")
@@
 	)
 	(segment
-		(start -3.5078 4.7178)
-		(end -4.8 4.7178)
+		(start 4.2 22.317014)
+		(end 4.2 18.27)
 		(width 0.25)
 		(layer "F.Cu")
@@
 	)
 	(segment
+		(start 2.9925 22.5925)
+		(end 3.924514 22.5925)
+		(width 0.25)
+		(layer "F.Cu")
+		(net 1)
+	)
+	(segment
 		(start -5.281846 6.015804)
 		(end -4.847129 6.450521)
@@
 	)
 	(segment
-		(start -2.906846 5.5178)
-		(end -2.906846 11.163154)
+		(start 2.55 20.3175)
+		(end 2.55 22.15)
 		(width 0.25)
 		(layer "F.Cu")
@@
 	)
 	(segment
-		(start 3.93 22.79)
-		(end 4.32 22.4)
+		(start 3.924514 22.5925)
+		(end 4.2 22.317014)
 		(width 0.25)
 		(layer "F.Cu")
@@
 	)
 	(segment
-		(start 3.12 22.74)
-		(end 3.17 22.79)
+		(start 4.2 18.27)
+		(end -2.906846 11.163154)
 		(width 0.25)
 		(layer "F.Cu")
@@
 	)
 	(segment
-		(start 4.32 22.4)
-		(end 4.38 22.34)
-		(width 0.25)
-		(layer "F.Cu")
-		(net 1)
-	)
-	(segment
-		(start 3.23 22.61)
-		(end 2.55 21.93)
+		(start -2.906846 11.163154)
+		(end -2.906846 5.5178)
 		(width 0.25)
 		(layer "F.Cu")
@@
 	)
 	(segment
-		(start 2.55 22.17)
-		(end 3.12 22.74)
-		(width 0.25)
-		(layer "F.Cu")
-		(net 1)
-	)
-	(segment
 		(start 2.55 17.892792)
 		(end -3.806846 11.535946)
@@
 	)
 	(segment
-		(start 4.2 18.27)
-		(end 4.2 22.317014)
-		(width 0.25)
-		(layer "F.Cu")
-		(net 1)
-	)
-	(segment
 		(start 2.55 20.3175)
 		(end 2.55 17.892792)
@@
 	)
 	(segment
-		(start 4.2 22.317014)
-		(end 3.907014 22.61)
-		(width 0.25)
-		(layer "F.Cu")
-		(net 1)
-	)
-	(segment
 		(start 2.55 20.3175)
 		(end 2.55 22.17)
@@
 	)
 	(segment
-		(start 3.907014 22.61)
-		(end 3.23 22.61)
+		(start 2.55 22.15)
+		(end 2.9925 22.5925)
 		(width 0.25)
 		(layer "F.Cu")
@@
 	)
 	(segment
-		(start 4.38 22.34)
-		(end 4.38 20.84)
-		(width 0.25)
-		(layer "F.Cu")
-		(net 1)
-	)
-	(segment
 		(start -4.847129 6.450521)
 		(end -4.54 6.450521)
@@
 	)
 	(segment
-		(start -2.906846 11.163154)
-		(end 4.2 18.27)
-		(width 0.25)
-		(layer "F.Cu")
-		(net 1)
-	)
-	(segment
-		(start 2.55 21.93)
-		(end 2.55 20.3175)
-		(width 0.25)
-		(layer "F.Cu")
-		(net 1)
-	)
-	(segment
-		(start 1.53 20.3175)
-		(end 1.53 18.11)
-		(width 0.5)
-		(layer "F.Cu")
-		(net 2)
-	)
-	(segment
 		(start -0.51 20.3175)
 		(end -0.51 17.86)
@@
 	)
 	(segment
-		(start 1.53 18.11)
-		(end 0.45 17.03)
-		(width 0.5)
-		(layer "F.Cu")
-		(net 2)
-	)
-	(segment
 		(start -24.24 1.6249)
 		(end -24.7451 2.13)
@@
 	)
 	(segment
+		(start 0.51 22.2675)
+		(end 1.817379 23.574879)
+		(width 0.5)
+		(layer "F.Cu")
+		(net 5)
+	)
+	(segment
+		(start 1.817379 23.574879)
+		(end 4.134879 23.574879)
+		(width 0.5)
+		(layer "F.Cu")
+		(net 5)
+	)
+	(segment
+		(start 5.09 22.619758)
+		(end 5.09 17.9)
+		(width 0.5)
+		(layer "F.Cu")
+		(net 5)
+	)
+	(segment
+		(start -2.02 10.79)
+		(end -2.02 6.85)
+		(width 0.5)
+		(layer "F.Cu")
+		(net 5)
+	)
+	(segment
+		(start -2.02 6.85)
+		(end 1.45 3.38)
+		(width 0.5)
+		(layer "F.Cu")
+		(net 5)
+	)
+	(segment
+		(start 5.09 17.9)
+		(end -2.02 10.79)
+		(width 0.5)
+		(layer "F.Cu")
+		(net 5)
+	)
+	(segment
+		(start 0.51 20.3175)
+		(end 0.51 22.2675)
+		(width 0.5)
+		(layer "F.Cu")
+		(net 5)
+	)
+	(segment
+		(start 4.134879 23.574879)
+		(end 5.09 22.619758)
+		(width 0.5)
+		(layer "F.Cu")
+		(net 5)
+	)
+	(segment
 		(start -3.38 -2.9)
 		(end -3.14 -3.14)
@@
 	)
 	(segment
+		(start -5.22 7.33)
+		(end -6.17 6.38)
+		(width 0.5)
+		(layer "F.Cu")
+		(net 9)
+	)
+	(segment
+		(start 1.53 18.11)
+		(end -4.69 11.89)
+		(width 0.5)
+		(layer "F.Cu")
+		(net 9)
+	)
+	(segment
 		(start -32.1802 1.805)
 		(end -33.81 1.805)
@@
 	)
 	(segment
+		(start -6.17 4.66)
+		(end -4.65 3.14)
+		(width 0.5)
+		(layer "F.Cu")
+		(net 9)
+	)
+	(segment
+		(start -4.69 11.89)
+		(end -4.69 7.33)
+		(width 0.5)
+		(layer "F.Cu")
+		(net 9)
+	)
+	(segment
+		(start -4.69 7.33)
+		(end -5.22 7.33)
+		(width 0.5)
+		(layer "F.Cu")
+		(net 9)
+	)
+	(segment
+		(start -6.17 6.38)
+		(end -6.17 4.66)
+		(width 0.5)
+		(layer "F.Cu")
+		(net 9)
+	)
+	(segment
+		(start 1.53 20.3175)
+		(end 1.53 18.11)
+		(width 0.5)
+		(layer "F.Cu")
+		(net 9)
+	)
+	(segment
+		(start -4.65 3.14)
+		(end -3.14 3.14)
+		(width 0.5)
+		(layer "F.Cu")
+		(net 9)
+	)
+	(segment
 		(start -4.23 21.82)
 		(end -5.04 22.63)
@@
 	(zone
 		(net 9)
-		(net_name "Net-(IC1-SET)")
+		(net_name "/LED+")
 		(layer "F.Cu")
 		(hatch edge 0.5)
@@
 	(zone
 		(net 5)
-		(net_name "Net-(D2-PAD)")
+		(net_name "/LED-")
 		(layer "F.Cu")
 		(hatch edge 0.5)
