File: KiCAD/LED Controller/LED controller.kicad_pcb (KiCad board)
At the start: 2 copper layers, 100 x 100 mm, 45 parts, among them J1 Barrel_Jack_Switch, J2 4x RJ45, J5 8P8C_Shielded, J6 Conn_01x03_Socket, J7 Conn_01x02_Socket, SW1 ELUMOASAQ2C22, SW2 ELUMOASAQ2C22, SW3 ELUMOASAQ2C22, U1 SN75374D, U2 SN75374D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

Commit message: Minor changes - ground strip along RJ45 12V, add part # for I2C socket
Routing:
- net GND: track 646.7 -> 681.0 mm
Other:
- board text added: "Digital Inputs -15V/+18V Max"
- board text removed: "Digital Inputs -14V/+17V Max"
Changed lines of the file:
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@@
 		(tags "capacitor")
 		(property "Reference" "C2"
-			(at 0 -1.43 360)
+			(at 0 -1.43 0)
 			(layer "F.SilkS")
 			(effects
@@
 		)
 		(property "Value" "1µF"
-			(at 0 1.43 360)
+			(at 0 1.43 0)
 			(layer "F.Fab")
 			(effects
@@
 		)
 		(fp_text user "${REFERENCE}"
-			(at 0 0 360)
+			(at 0 0 0)
 			(layer "F.Fab")
 			(effects
@@
 		(tags "capacitor")
 		(property "Reference" "C7"
-			(at -2.21 -0.2 360)
+			(at -2.21 -0.2 0)
 			(layer "F.SilkS")
 			(effects
@@
 		(tags "capacitor")
 		(property "Reference" "C6"
-			(at -2.24 0.08 360)
+			(at -2.24 0.08 0)
 			(layer "F.SilkS")
 			(effects
@@
 		(tags "capacitor")
 		(property "Reference" "C11"
-			(at 0.04 1.48 360)
+			(at 0.04 1.48 0)
 			(layer "F.SilkS")
 			(effects
@@
 		)
 		(property "Value" "1µF"
-			(at 0 1.43 360)
+			(at 0 1.43 0)
 			(layer "F.Fab")
 			(effects
@@
 		)
 		(fp_text user "${REFERENCE}"
-			(at 0 0 360)
+			(at 0 0 0)
 			(layer "F.Fab")
 			(effects
@@
 		(tags "capacitor")
 		(property "Reference" "C1"
-			(at 0 -1.43 360)
+			(at 0 -1.43 0)
 			(layer "F.SilkS")
 			(effects
@@
 		)
 		(property "Value" "1µF"
-			(at 0 1.43 360)
+			(at 0 1.43 0)
 			(layer "F.Fab")
 			(effects
@@
 		)
 		(fp_text user "${REFERENCE}"
-			(at 0 0 360)
+			(at 0 0 0)
 			(layer "F.Fab")
 			(effects
@@
 		)
 	)
-	(gr_text "Digital Inputs\n-14V/+17V Max"
+	(gr_text "Digital Inputs\n-15V/+18V Max"
 		(at 90.46 21 0)
 		(layer "F.SilkS")
@@
 	)
 	(segment
+		(start 54.815 16.605)
+		(end 56.4125 15.0075)
+		(width 0.2)
+		(layer "F.Cu")
+		(net 2)
+	)
+	(segment
 		(start 62.36 72.12)
 		(end 62.36 71.01)
@@
 	)
 	(segment
+		(start 53.265 15.9975)
+		(end 53.8725 16.605)
+		(width 0.2)
+		(layer "F.Cu")
+		(net 2)
+	)
+	(segment
 		(start 81.300735 59.640738)
 		(end 80.653342 60.288131)
@@
 	)
 	(segment
+		(start 66.4775 13.465)
+		(end 69.8325 16.82)
+		(width 0.2)
+		(layer "F.Cu")
+		(net 2)
+	)
+	(segment
 		(start 71.4275 15.075)
 		(end 71.4275 14.085)
@@
 	)
 	(segment
+		(start 56.4125 13.6825)
+		(end 56.63 13.465)
+		(width 0.2)
+		(layer "F.Cu")
+		(net 2)
+	)
+	(segment
 		(start 73.303342 62.2272)
 		(end 73.276142 62.2)
@@
 	)
 	(segment
+		(start 41.7875 13.505)
+		(end 53.265 13.505)
+		(width 0.2)
+		(layer "F.Cu")
+		(net 2)
+	)
+	(segment
 		(start 72.073942 65.681744)
 		(end 72.04 65.715686)
@@
 	)
 	(segment
+		(start 56.63 13.465)
+		(end 66.4775 13.465)
+		(width 0.2)
+		(layer "F.Cu")
+		(net 2)
+	)
+	(segment
 		(start 81.83 57.697256)
 		(end 81.83 57.27)
@@
 	)
 	(segment
+		(start 53.265 13.505)
+		(end 53.265 15.9975)
+		(width 0.2)
+		(layer "F.Cu")
+		(net 2)
+	)
+	(segment
 		(start 28.439986 20.01725)
 		(end 28.439986 19.398542)
@@
 	)
 	(segment
+		(start 53.8725 16.605)
+		(end 54.815 16.605)
+		(width 0.2)
+		(layer "F.Cu")
+		(net 2)
+	)
+	(segment
 		(start 79.887657 59.639599)
 		(end 81.83 57.697256)
@@
 		(layer "F.Cu")
 		(net 2)
+	)
+	(segment
+		(start 56.4125 15.0075)
+		(end 56.4125 13.6825)
+		(width 0.2)
+		(layer "F.Cu")
+		(net 2)

Commit message: Label schematic - switch to 10-bit DAC
Parts:
- U1, U2, U3: value SN75374D -> 4x Gate Driver
- U5: value SN74LV4053ADR -> 3x Analog Switch
- U6: value DAC084S085CIMMX/NOPB -> 3x 10-Bit DAC
- U7: value NXB0104PWJ -> 3x Level Shifter
Changed lines of the file:
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@@
 			)
 		)
-		(property "Value" "SN75374D"
+		(property "Value" "4x Gate Driver"
 			(at 0 0 90)
 			(unlocked yes)
@@
 			)
 		)
-		(property "Value" "NXB0104PWJ"
+		(property "Value" "3x Level Shifter"
 			(at 0 0 90)
 			(unlocked yes)
@@
 			)
 		)
-		(property "Value" "SN75374D"
+		(property "Value" "4x Gate Driver"
 			(at 0 0 90)
 			(unlocked yes)
@@
 			)
 		)
-		(property "Part" "P160KN2-4QC20B10K"
+		(property "Part" "P160KN2-0QA25B10K"
 			(at 0 0 0)
 			(unlocked yes)
@@
 			)
 		)
-		(property "Value" "DAC084S085CIMMX/NOPB"
+		(property "Value" "3x 10-Bit DAC"
 			(at 0 0 180)
 			(unlocked yes)
@@
 			)
 		)
-		(property "Datasheet" "https://www.ti.com/general/docs/suppproductinfo.tsp?distId=10&gotoUrl=https%3A%2F%2Fwww.ti.com%2Flit%2Fgpn%2Fdac084s085"
+		(property "Datasheet" "https://www.ti.com/lit/ds/symlink/dac104s085-q1.pdf"
 			(at 0 0 0)
 			(layer "F.Fab")
@@
 			)
 		)
-		(property "Description" "IC DAC 8BIT V-OUT 10VSSOP"
+		(property "Description" "IC DAC 10BIT V-OUT 10VSSOP"
 			(at 0 0 0)
 			(layer "F.Fab")
@@
 			)
 		)
-		(property "Part" "DAC084S085CIMMX/NOPB"
+		(property "Part" "DAC104S085QIMMX/NOPB"
 			(at 0 0 180)
 			(unlocked yes)
@@
 			)
 		)
-		(property "Value" "SN74LV4053ADR"
+		(property "Value" "3x Analog Switch"
 			(at 0 0 -90)
 			(unlocked yes)
@@
 			)
 		)
-		(property "Part" "P160KN2-4QC20B10K"
+		(property "Part" "P160KN2-0QA25B10K"
 			(at 0 0 0)
 			(unlocked yes)
@@
 			)
 		)
-		(property "Value" "SN75374D"
+		(property "Value" "4x Gate Driver"
 			(at 0 0 90)
 			(unlocked yes)
@@
 			)
 		)
-		(property "Part" "P160KN2-4QC20B10K"
+		(property "Part" "P160KN2-0QA25B10K"
 			(at 0 0 0)
 			(unlocked yes)
@@
 			)
 		)
-		(property "Datasheet" ""
+		(property "Datasheet" "https://app.adam-tech.com/products/download/data_sheet/203013/rs1-xx-g-data-sheet.pdf"
 			(at 0 0 90)
 			(unlocked yes)
@@
 			)
 		)
-		(property "Description" "Generic connector, single row, 01x02, script generated"
+		(property "Description" "RECEPTACLE STRIP 2P 2.54MM PITCH"
 			(at 0 0 90)
 			(unlocked yes)
@@
 			)
 		)
-		(property "Manufacturer" ""
+		(property "Manufacturer" "Adam Tech"
 			(at 0 0 90)
 			(unlocked yes)
@@
 			)
 		)
-		(property "Part" ""
+		(property "Part" "RS1-02-G"
 			(at 0 0 90)
 			(unlocked yes)
